File: mcu.kicad_sch (KiCad schematic)
At the start: 12 parts, among them U1 STM32G0B1CBU6, Y1 SC32S-7PF20PPM

Commit message: Initial layout
Connections:
- net BACKLIGHT: now also U1.14 (PA3); no longer U1.22 (PB10)
- net BUTTON: now also U1.1 (PC13); no longer U1.27 (PB15)
- net BUZZER: now also U1.47 (PB8); no longer U1.26 (PB14)
- net DISPLAY.A0: now also U1.17 (PA6); no longer U1.20 (PB1)
- net DISPLAY.CS: now also U1.20 (PB1); no longer U1.17 (PA6)
- net KEY0: now also U1.25 (PB13); no longer U1.44 (PB5)
- net KEY1: now also U1.26 (PB14); no longer U1.43 (PB4)
- net KEY2: now also U1.27 (PB15); no longer U1.42 (PB3)
- net KEY3: now also U1.13 (PA2); no longer U1.41 (PD3)
- net LED: now also U1.48 (PB9); no longer U1.25 (PB13)
- net LIS2_INT: now also U1.43 (PB4); no longer U1.47 (PB8)
- net MIC: now also U1.24 (PB12); no longer U1.14 (PA3)
- net SW_PWR_EN: now also U1.37 (PA15); no longer U1.13 (PA2)
- net VL53_EN: now also U1.44 (PB5); no longer U1.48 (PB9)
Other:
- note added: "ADC_IN16"
- note added: "TIM16_CH1"
- note removed: "ADC_IN3"
- note removed: "TIM15_CH1"
