File: Puzzlebox-HW.kicad_pcb (KiCad board)
At the start: 4 copper layers, 50 x 50 mm, 107 parts, among them J1 USB4145-03-0170-C, J2 B2B-PH-K-S, J3 S2B-PH-K-S, J4 SFV31R-4STE1HLF, J5 F3311A7H121004E200, J6 F3311A7H121004E200, J7 F3311A7H121004E200, J8 F3311A7H121004E200, M1 Mount_M3, M2 Mount_M3, M3 Mount_M3, M4 Mount_M3, Q1 DMG1012UW-7, Q2 DMG1013UW-7, Q3 DMG1012UW-7, Q4 DMG1012UW-7, Q5 DMG1012UW-7, Q6 DMG1012UW-7, U1 STM32G0B1CBU6, U10 BME280, U11 VEML3328, U12 ICS-40212, U13 SMT-0827-S-HT-R, U14 TLV9041IDBVR, U15 AT42QT1010-TSHR, U16 AT42QT1010-TSHR, U17 AT42QT1010-TSHR, U18 AT42QT1010-TSHR, U2 USBLC6-4SC6, U3 MCP73832T-2ACI/OT, U4 MCP1711T-30I/OT, U5 MCP1711T-30I/OT, U6 LIS2DTW12TR, U7 24FC512T-I/OT, U8 LIS2MDLTR, U9 VL53L4CXV0DH/1, Y1 SC32S-7PF20PPM

Commit message: Add some notes. Configure outputs.
Parts:
- moved FID2 35.5 mm to (93.5, 60.4)
Changed lines of the file:
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@@
 			(layer "F.SilkS"
 				(type "Top Silk Screen")
+				(color "White")
 			)
 			(layer "F.Paste"
@@
 			(layer "F.Mask"
 				(type "Top Solder Mask")
+				(color "Purple")
 				(thickness 0.01)
 			)
@@
 			(layer "B.Mask"
 				(type "Bottom Solder Mask")
+				(color "Purple")
 				(thickness 0.01)
 			)
@@
 			(layer "B.SilkS"
 				(type "Bottom Silk Screen")
+				(color "White")
 			)
 			(copper_finish "None")
@@
 		(at 88.9 52.4)
 		(property "Reference" "J2"
-			(at 2.35 4 180)
+			(at 1.75 3.85 180)
 			(layer "F.SilkS")
 			(effects
@@
 	(footprint "N_NonPart:Fiducial_2mm"
 		(layer "F.Cu")
-		(at 58.2 56.4)
+		(at 93.45 60.35)
 		(property "Reference" "FID2"
 			(at 0 -2.3 0)
