File: display.kicad_sch (KiCad schematic)
At the start: 9 parts, among them J3 S2B-PH-K-S, J4 SFV31R-4STE1HLF, Q3 DMG1012UW-7

Commit message: Initial layout
Connections:
- net +3V0_SW: now also J4.12, J4.13, J4.14, J4.15, J4.30; no longer J4.17, J4.18, J4.19, J4.2, J4.20
- net DISPLAY.A0: now also J4.26; no longer J4.6
- net DISPLAY.CS: now also J4.28; no longer J4.4
- net DISPLAY.RST: now also J4.27; no longer J4.5
- net DISPLAY.SCK: now also J4.17; no longer J4.15
- net GND: now also J4.10, J4.11, J4.29, J4.31, J4.8, J4.9; no longer J4.1, J4.21, J4.22, J4.23, J4.24, J4.3
- net at C12.1: now also J4.5; no longer J4.27
- net at C13.1: now also J4.4; no longer J4.28
Changed lines of the file:
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@@
-	(wire
-		(pts
-			(xy 190.5 116.84) (xy 190.5 121.92)
-		)
-		(stroke
-			(width 0)
-			(type default)
-		)
-	)
 	(wire
 		(pts
@@
 	(wire
 		(pts
-			(xy 187.96 116.84) (xy 190.5 116.84)
-		)
-		(stroke
-			(width 0)
-			(type default)
-		)
-	)
-	(wire
-		(pts
 			(xy 162.56 40.64) (xy 175.26 40.64)
 		)
@@
 	(wire
 		(pts
+			(xy 189.23 40.64) (xy 189.23 121.92)
+		)
+		(stroke
+			(width 0)
+			(type default)
+		)
+	)
+	(wire
+		(pts
 			(xy 144.78 53.34) (xy 175.26 53.34)
 		)
@@
 	(wire
 		(pts
-			(xy 162.56 121.92) (xy 190.5 121.92)
+			(xy 162.56 121.92) (xy 189.23 121.92)
 		)
 		(stroke
@@
 		(pts
 			(xy 204.47 92.71) (xy 204.47 95.25)
+		)
+		(stroke
+			(width 0)
+			(type default)
+		)
+	)
+	(wire
+		(pts
+			(xy 187.96 40.64) (xy 189.23 40.64)
 		)
 		(stroke
@@
 	(symbol
 		(lib_id "lib:SFV31R-4STE1HLF")
-		(at 181.61 119.38 0)
+		(at 181.61 38.1 0)
+		(mirror x)
 		(unit 1)
 		(exclude_from_sim no)
@@
 		)
 		(property "Footprint" "lib:SFV31R-4STE1HLF"
-			(at 180.34 -13.97 0)
+			(at 180.34 171.45 0)
 			(effects
 				(font
@@
 		)
 		(property "Datasheet" "https://cdn.amphenol-cs.com/media/wysiwyg/files/documentation/datasheet/flex/flexconnectors_050mm_sfvr.pdf"
-			(at 181.61 124.46 0)
+			(at 181.61 33.02 0)
 			(effects
 				(font
@@
 		)
 		(property "Description" "CONN FPC TOP 31POS 0.5MM R/A"
-			(at 181.356 127 0)
-			(effects
-				(font
+			(at 181.356 30.48 0)
+			(effects
+				(font

Commit message: Add some notes. Configure outputs.
Other:
- moved on the sheet: J3, Q3, R10, R9
Changed lines of the file:
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@@
 		)
 	)
-	(text_box "Display: 2.2\" 128x128 LCD\nController: ST7571\nPN: ERC128128FS02-3"
+	(text_box "FFC Connector to display\nDisplay: 2.2\" 128x128 LCD\nController: ST7571\nPN: ERC128128FS02-3"
 		(exclude_from_sim no)
 		(at 203.2 43.18 0)
-		(size 40.64 7.62)
+		(size 30.48 10.16)
+		(margins 0.9525 0.9525 0.9525 0.9525)
+		(stroke
+			(width 0)
+			(type solid)
+		)
+		(fill
+			(type none)
+		)
+		(effects
+			(font
+				(size 1.27 1.27)
+			)
+			(justify left top)
+		)
+	)
+	(text_box "Backlight connector"
+		(exclude_from_sim no)
+		(at 95.25 87.63 0)
+		(size 21.59 3.81)
 		(margins 0.9525 0.9525 0.9525 0.9525)
 		(stroke
@@
 	)
 	(junction
-		(at 86.36 123.19)
+		(at 69.85 123.19)
 		(diameter 0)
 		(color 0 0 0 0)
@@
 	)
 	(junction
-		(at 74.93 111.76)
+		(at 58.42 111.76)
 		(diameter 0)
 		(color 0 0 0 0)
@@
 	(wire
 		(pts
-			(xy 86.36 101.6) (xy 86.36 106.68)
+			(xy 69.85 101.6) (xy 69.85 106.68)
 		)
 		(stroke
@@
 	(wire
 		(pts
-			(xy 88.9 87.63) (xy 86.36 87.63)
+			(xy 72.39 87.63) (xy 69.85 87.63)
 		)
 		(stroke
@@
 	(wire
 		(pts
-			(xy 86.36 116.84) (xy 86.36 123.19)
-		)
-		(stroke
-			(width 0)
-			(type default)
-		)
-	)
-	(wire
-		(pts
-			(xy 86.36 123.19) (xy 86.36 124.46)
-		)
-		(stroke
-			(width 0)
-			(type default)
-		)
-	)
-	(wire
-		(pts
-			(xy 86.36 83.82) (xy 86.36 87.63)
-		)
-		(stroke
-			(width 0)
-			(type default)
-		)
-	)
-	(wire
-		(pts
-			(xy 74.93 123.19) (xy 86.36 123.19)
-		)
-		(stroke
-			(width 0)
-			(type default)
-		)
-	)
-	(wire
-		(pts
-			(xy 74.93 114.3) (xy 74.93 111.76)
-		)
-		(stroke
-			(width 0)
-			(type default)
-		)
-	)
-	(wire
-		(pts
-			(xy 74.93 111.76) (xy 81.28 111.76)
+			(xy 69.85 116.84) (xy 69.85 123.19)
+		)
+		(stroke
+			(width 0)
+			(type default)
+		)
+	)
+	(wire
+		(pts
+			(xy 69.85 123.19) (xy 69.85 124.46)
+		)
+		(stroke
+			(width 0)
+			(type default)
+		)
+	)
+	(wire
+		(pts
+			(xy 69.85 83.82) (xy 69.85 87.63)
+		)
+		(stroke
+			(width 0)
+			(type default)
+		)
+	)
+	(wire
+		(pts
+			(xy 58.42 123.19) (xy 69.85 123.19)
+		)
+		(stroke
+			(width 0)
+			(type default)
+		)
+	)
+	(wire
+		(pts
+			(xy 58.42 114.3) (xy 58.42 111.76)
+		)
+		(stroke
+			(width 0)
+			(type default)
+		)
+	)
+	(wire
+		(pts
+			(xy 58.42 111.76) (xy 64.77 111.76)
 		)
 		(stroke
@@
 	(wire
 		(pts
-			(xy 86.36 90.17) (xy 86.36 96.52)
+			(xy 69.85 90.17) (xy 69.85 96.52)
 		)
 		(stroke
@@
 	(wire
 		(pts
-			(xy 86.36 90.17) (xy 88.9 90.17)
-		)
-		(stroke
-			(width 0)
-			(type default)
-		)
-	)
-	(wire
-		(pts
-			(xy 67.31 111.76) (xy 74.93 111.76)
+			(xy 69.85 90.17) (xy 72.39 90.17)
+		)
+		(stroke
+			(width 0)
+			(type default)
+		)
+	)
+	(wire
+		(pts
+			(xy 50.8 111.76) (xy 58.42 111.76)
 		)
 		(stroke
@@
 	(wire
 		(pts
-			(xy 74.93 119.38) (xy 74.93 123.19)
+			(xy 58.42 119.38) (xy 58.42 123.19)
 		)
 		(stroke
@@
 	(hierarchical_label "BACKLIGHT"
 		(shape input)
-		(at 67.31 111.76 180)
+		(at 50.8 111.76 180)
 		(effects
 			(font
@@
 	(symbol
 		(lib_id "J_Connector:S2B-PH-K-S")
-		(at 92.71 86.36 0)
+		(at 76.2 86.36 0)
 		(mirror x)
 		(unit 1)
@@
 		(fields_autoplaced yes)
 		(property "Reference" "J3"
-			(at 95.25 87.6299 0)
+			(at 78.74 87.6299 0)
 			(effects
 				(font
@@
 		)
 		(property "Value" "S2B-PH-K-S"
-			(at 95.25 90.1699 0)
+			(at 78.74 90.1699 0)
 			(effects
 				(font
@@
 		)
 		(property "Footprint" "J_Connector:JST-S2B-PH-K-S"
-			(at 92.71 83.185 0)
+			(at 76.2 83.185 0)
 			(effects
 				(font
@@
 		)
 		(property "Datasheet" "https://www.jst-mfg.com/product/pdf/eng/ePH.pdf"
-			(at 92.71 81.28 0)
+			(at 76.2 81.28 0)
 			(effects
 				(font
@@
 		)
 		(property "Description" "CONN HEADER R/A 2POS 2MM"
-			(at 92.964 78.994 0)
+			(at 76.454 78.994 0)
 			(effects
 				(font
@@
 	(symbol
 		(lib_id "R_Resistor:R_0603")
-		(at 86.36 99.06 0)
+		(at 69.85 99.06 0)
 		(mirror y)
 		(unit 1)
@@
 		(fields_autoplaced yes)
 		(property "Reference" "R10"
-			(at 88.9 97.1549 0)
+			(at 72.39 97.1549 0)
 			(effects
 				(font
@@
 		)
 		(property "Value" "22R"
-			(at 88.9 99.6949 0)
+			(at 72.39 99.6949 0)
 			(effects
 				(font
@@
 		)
 		(property "Footprint" "R_Resistor:R_0603"
-			(at 88.9 99.06 90)
+			(at 72.39 99.06 90)
 			(effects
 				(font
@@
 		)
 		(property "Datasheet" ""
-			(at 88.9 102.87 0)
+			(at 72.39 102.87 0)
 			(effects
 				(font
@@
 		)
 		(property "Description" ""
-			(at 86.36 99.06 0)
+			(at 69.85 99.06 0)
 			(effects
 				(font
@@
 		)
 		(property "Size" "R_0603"
-			(at 88.9 101.6 0)
+			(at 72.39 101.6 0)
 			(effects
 				(font
@@
 	(symbol
 		(lib_id "R_Resistor:R_0603")
-		(at 74.93 116.84 0)
+		(at 58.42 116.84 0)
 		(mirror y)
 		(unit 1)
@@
 		(fields_autoplaced yes)
 		(property "Reference" "R9"
-			(at 77.47 114.9349 0)
+			(at 60.96 114.9349 0)
 			(effects
 				(font
@@
 		)
 		(property "Value" "100K"
-			(at 77.47 117.4749 0)
+			(at 60.96 117.4749 0)
 			(effects
 				(font
@@
 		)
 		(property "Footprint" "R_Resistor:R_0603"
-			(at 77.47 116.84 90)
+			(at 60.96 116.84 90)
 			(effects
 				(font
@@
 		)
 		(property "Datasheet" ""
-			(at 77.47 120.65 0)
+			(at 60.96 120.65 0)
 			(effects
 				(font
@@
 		)
 		(property "Description" ""
-			(at 74.93 116.84 0)
+			(at 58.42 116.84 0)
 			(effects
 				(font
@@
 		)
 		(property "Size" "R_0603"
-			(at 77.47 119.38 0)
+			(at 60.96 119.38 0)
 			(effects
 				(font
@@
 	(symbol
 		(lib_id "power:+BATT")
-		(at 86.36 83.82 0)
+		(at 69.85 83.82 0)
 		(unit 1)
 		(exclude_from_sim no)
@@
 		(fields_autoplaced yes)
 		(property "Reference" "#PWR024"
-			(at 86.36 87.63 0)
+			(at 69.85 87.63 0)
 			(effects
 				(font
@@
 		)
 		(property "Value" "+BATT"
-			(at 86.36 78.74 0)
+			(at 69.85 78.74 0)
 			(effects
 				(font
@@
 		)
 		(property "Footprint" ""
-			(at 86.36 83.82 0)
+			(at 69.85 83.82 0)
 			(effects
 				(font
@@
 		)
 		(property "Datasheet" ""
-			(at 86.36 83.82 0)
+			(at 69.85 83.82 0)
 			(effects
 				(font
@@
 		)
 		(property "Description" "Power symbol creates a global label with name \"+BATT\""
-			(at 86.36 83.82 0)
+			(at 69.85 83.82 0)
 			(effects
 				(font
@@
 	(symbol
 		(lib_id "Q_MOSFET:DMG1012UW-7")
-		(at 86.36 111.76 0)
+		(at 69.85 111.76 0)
 		(unit 1)
 		(exclude_from_sim no)
@@
 		(fields_autoplaced yes)
 		(property "Reference" "Q3"
-			(at 88.9 110.4899 0)
+			(at 72.39 110.4899 0)
 			(effects
 				(font
@@
 		)
 		(property "Value" "DMG1012UW-7"
-			(at 88.9 113.0299 0)
+			(at 72.39 113.0299 0)
 			(effects
 				(font
@@
 		)
 		(property "Footprint" "U_IC:SC70-3"
-			(at 86.36 127 0)
+			(at 69.85 127 0)
 			(effects
 				(font
@@
 		)
 		(property "Datasheet" "https://www.diodes.com/assets/Datasheets/DMG1012UW.pdf"
-			(at 85.09 124.46 0)
+			(at 68.58 124.46 0)
 			(effects
 				(font
@@
 		)
 		(property "Description" "MOSFET N-CH 20V 1A SOT323"
-			(at 86.36 129.286 0)
+			(at 69.85 129.286 0)
 			(effects
 				(font
@@
 	(symbol
 		(lib_id "power:GND")
-		(at 86.36 124.46 0)
+		(at 69.85 124.46 0)
 		(unit 1)
 		(exclude_from_sim no)
@@
 		(fields_autoplaced yes)
 		(property "Reference" "#PWR025"
-			(at 86.36 130.81 0)
+			(at 69.85 130.81 0)
 			(effects
 				(font
@@
 		)
 		(property "Value" "GND"
-			(at 86.36 129.54 0)
+			(at 69.85 129.54 0)
 			(effects
 				(font
@@
 		)
 		(property "Footprint" ""
-			(at 86.36 124.46 0)
+			(at 69.85 124.46 0)
 			(effects
 				(font
@@
 		)
 		(property "Datasheet" ""
-			(at 86.36 124.46 0)
+			(at 69.85 124.46 0)
 			(effects
 				(font
@@
 		)
 		(property "Description" "Power symbol creates a global label with name \"GND\" , ground"
-			(at 86.36 124.46 0)
-			(effects
-				(font
+			(at 69.85 124.46 0)
+			(effects
+				(font
