File: power.kicad_sch (KiCad schematic)
At the start: 21 parts, among them J1 USB4145-03-0170-C, J2 B2B-PH-K-S, Q1 DMG1012UW-7, Q2 DMG1013UW-7, U2 USBLC6-4SC6, U3 MCP73832T-2ACI/OT, U4 MCP1711T-30I/OT, U5 MCP1711T-30I/OT

Commit message: Initial layout
Connections:
- net +BATT: now also Q2.2 (S); no longer Q2.3 (D)
- net USB.CC1: now also U2.3; no longer U2.1
- net USB.CC2: now also U2.1; no longer U2.3
- net USB.DM: now also U2.6; no longer U2.4
- net USB.DP: now also U2.4; no longer U2.6
- net at R5.2: now also Q2.3 (D); no longer Q2.2 (S)
Changed lines of the file:
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@@
 	)
 	(junction
-		(at 106.68 76.2)
-		(diameter 0)
-		(color 0 0 0 0)
-	)
-	(junction
-		(at 104.14 78.74)
+		(at 82.55 68.58)
+		(diameter 0)
+		(color 0 0 0 0)
+	)
+	(junction
+		(at 80.01 66.04)
 		(diameter 0)
 		(color 0 0 0 0)
@@
 	)
 	(junction
-		(at 82.55 66.04)
-		(diameter 0)
-		(color 0 0 0 0)
-	)
-	(junction
-		(at 80.01 68.58)
-		(diameter 0)
-		(color 0 0 0 0)
-	)
-	(junction
 		(at 199.39 134.62)
 		(diameter 0)
@@
 	)
 	(junction
+		(at 104.14 76.2)
+		(diameter 0)
+		(color 0 0 0 0)
+	)
+	(junction
 		(at 69.85 101.6)
 		(diameter 0)
@@
 	(junction
 		(at 199.39 92.71)
+		(diameter 0)
+		(color 0 0 0 0)
+	)
+	(junction
+		(at 106.68 78.74)
 		(diameter 0)
 		(color 0 0 0 0)
@@
 	(wire
 		(pts
+			(xy 80.01 66.04) (xy 111.76 66.04)
+		)
+		(stroke
+			(width 0)
+			(type default)
+		)
+	)
+	(wire
+		(pts
 			(xy 161.29 45.72) (xy 161.29 50.8)
 		)
@@
 	(wire
 		(pts
+			(xy 106.68 78.74) (xy 111.76 78.74)
+		)
+		(stroke
+			(width 0)
+			(type default)
+		)
+	)
+	(wire
+		(pts
 			(xy 199.39 119.38) (xy 199.39 127)
 		)
@@
 	(wire
 		(pts
-			(xy 80.01 95.25) (xy 80.01 68.58)
-		)
-		(stroke
-			(width 0)
-			(type default)
-		)
-	)
-	(wire
-		(pts
 			(xy 63.5 53.34) (xy 69.85 53.34)
 		)
@@
 	(wire
 		(pts
-			(xy 104.14 78.74) (xy 111.76 78.74)
+			(xy 66.04 78.74) (xy 106.68 78.74)
 		)
 		(stroke
@@
 	(wire
 		(pts
-			(xy 82.55 66.04) (xy 111.76 66.04)
+			(xy 63.5 66.04) (xy 80.01 66.04)
 		)
 		(stroke
@@
 	(wire
 		(pts
-			(xy 63.5 68.58) (xy 80.01 68.58)
-		)
-		(stroke
-			(width 0)
-			(type default)
-		)
-	)
-	(wire
-		(pts
-			(xy 66.04 78.74) (xy 104.14 78.74)
-		)
-		(stroke
-			(width 0)
-			(type default)
-		)
-	)
-	(wire
-		(pts
 			(xy 96.52 166.37) (xy 96.52 168.91)
 		)
@@
 	(wire
 		(pts
-			(xy 106.68 95.25) (xy 106.68 76.2)
-		)
-		(stroke
-			(width 0)
-			(type default)
-		)
-	)
-	(wire
-		(pts
 			(xy 69.85 58.42) (xy 69.85 60.96)
 		)
@@
 	(wire
 		(pts
+			(xy 80.01 66.04) (xy 80.01 95.25)
+		)
+		(stroke
+			(width 0)
+			(type default)
+		)
+	)
+	(wire
+		(pts
 			(xy 199.39 81.28) (xy 199.39 85.09)
 		)
@@
 	(wire
 		(pts
-			(xy 66.04 76.2) (xy 106.68 76.2)
-		)
-		(stroke
-			(width 0)
-			(type default)
-		)
-	)
-	(wire
-		(pts
 			(xy 123.19 147.32) (xy 102.87 147.32)
 		)
@@
 	(wire
 		(pts
+			(xy 82.55 68.58) (xy 82.55 92.71)
+		)
+		(stroke
+			(width 0)
+			(type default)
+		)
+	)
+	(wire
+		(pts
 			(xy 128.27 166.37) (xy 128.27 168.91)
 		)
@@
 	(wire
 		(pts
+			(xy 82.55 68.58) (xy 111.76 68.58)
+		)
+		(stroke
+			(width 0)
+			(type default)
+		)
+	)
+	(wire
+		(pts
 			(xy 96.52 161.29) (xy 96.52 158.75)
 		)
@@
 	(wire
 		(pts
-			(xy 82.55 92.71) (xy 82.55 66.04)
-		)
-		(stroke
-			(width 0)
-			(type default)
-		)
-	)
-	(wire
-		(pts
-			(xy 80.01 68.58) (xy 111.76 68.58)
-		)
-		(stroke
-			(width 0)
-			(type default)
-		)
-	)
-	(wire
-		(pts
-			(xy 63.5 66.04) (xy 82.55 66.04)
+			(xy 104.14 76.2) (xy 111.76 76.2)
+		)
+		(stroke
+			(width 0)
+			(type default)
+		)
+	)
+	(wire
+		(pts
+			(xy 63.5 68.58) (xy 82.55 68.58)
 		)
 		(stroke
@@
 	(wire
 		(pts
-			(xy 104.14 92.71) (xy 104.14 78.74)
-		)
-		(stroke
-			(width 0)
-			(type default)
-		)
-	)
-	(wire
-		(pts
 			(xy 180.34 50.8) (xy 170.18 50.8)
 		)
@@
 	(wire
 		(pts
-			(xy 106.68 76.2) (xy 111.76 76.2)
+			(xy 106.68 78.74) (xy 106.68 95.25)
+		)
+		(stroke
+			(width 0)
+			(type default)
+		)
+	)
+	(wire
+		(pts
+			(xy 66.04 76.2) (xy 104.14 76.2)
 		)
 		(stroke
@@
 		(pts
 			(xy 128.27 137.16) (xy 128.27 138.43)
+		)
+		(stroke
+			(width 0)
+			(type default)
+		)
+	)
+	(wire
+		(pts
+			(xy 104.14 76.2) (xy 104.14 92.71)
 		)
 		(stroke
@@
 		(lib_id "Q_MOSFET:DMG1013UW-7")
 		(at 128.27 147.32 0)
+		(mirror x)
 		(unit 1)
 		(exclude_from_sim no)
@@
 		(on_board yes)
 		(dnp no)
-		(fields_autoplaced yes)
 		(property "Reference" "Q2"
-			(at 130.81 146.0499 0)
+			(at 130.81 148.5901 0)
 			(effects
 				(font
@@
 		)
 		(property "Value" "DMG1013UW-7"
-			(at 130.81 148.5899 0)
+			(at 130.81 146.0501 0)
 			(effects
 				(font
@@
 		)
 		(property "Footprint" "U_IC:SC70-3"
-			(at 128.27 162.56 0)
+			(at 128.27 132.08 0)
 			(effects
 				(font
@@
 		)
 		(property "Datasheet" "https://www.diodes.com/assets/Datasheets/ds31861.pdf"
-			(at 127 160.02 0)
+			(at 127 134.62 0)
 			(effects
 				(font
@@
 		)
 		(property "Description" "MOSFET P-CH 20V 820MA SOT323"
-			(at 128.524 164.846 0)
-			(effects
-				(font
+			(at 128.524 129.794 0)
+			(effects
+				(font

Commit message: Add some notes. Configure outputs.
Changed lines of the file:
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@@
 		(company "TL Embedded Ltd")
+	)
+	(text_box "1S Li-ion pack"
+		(exclude_from_sim no)
+		(at 252.73 31.75 0)
+		(size 17.78 3.81)
+		(margins 0.9525 0.9525 0.9525 0.9525)
+		(stroke
+			(width 0)
+			(type solid)
+		)
+		(fill
+			(type none)
+		)
+		(effects
+			(font
+				(size 1.27 1.27)
+			)
+			(justify left top)
+		)
 	)
 	(junction
