File: touch.kicad_sch (KiCad schematic)
At the start: 20 parts, among them J5 F3311A7H121004E200, J6 F3311A7H121004E200, J7 F3311A7H121004E200, J8 F3311A7H121004E200, U15 AT42QT1010-TSHR, U16 AT42QT1010-TSHR, U17 AT42QT1010-TSHR, U18 AT42QT1010-TSHR

Commit message: Initial layout
Connections:
- net KEY1: now also U16.1 (OUT); no longer U17.1 (OUT)
- net KEY2: now also U17.1 (OUT); no longer U16.1 (OUT)
Changed lines of the file:
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@@
+	)
+	(label "KEY1"
+		(at 43.18 85.09 0)
+		(effects
+			(font
+				(size 1.27 1.27)
+			)
+			(justify left bottom)
+		)
 	)
 	(label "KEY1"
@@
 		)
 	)
-	(label "KEY3"
-		(at 152.4 82.55 0)
+	(label "KEY2"
+		(at 152.4 38.1 0)
 		(effects
 			(font
@@
 		)
 	)
-	(label "KEY1"
-		(at 152.4 38.1 0)
+	(label "KEY3"
+		(at 152.4 82.55 0)
 		(effects
 			(font
@@
 		)
 	)
-	(label "KEY2"
-		(at 43.18 85.09 0)
-		(effects
-			(font
-				(size 1.27 1.27)
-			)
-			(justify left bottom)
-		)
-	)

Commit message: Add some notes. Configure outputs.
Changed lines of the file:
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@@
 		(company "TL Embedded Ltd")
+	)
+	(text_box "FFC connectors to touch panels"
+		(exclude_from_sim no)
+		(at 104.14 106.68 0)
+		(size 34.29 3.81)
+		(margins 0.9525 0.9525 0.9525 0.9525)
+		(stroke
+			(width 0)
+			(type solid)
+		)
+		(fill
+			(type none)
+		)
+		(effects
+			(font
+				(size 1.27 1.27)
+			)
+			(justify left top)
+		)
 	)
 	(junction
